File: Power.kicad_sch (KiCad schematic)
At the start: 9 parts, among them J901 Screw_Terminal_01x02, U901 AZ1117-3.3

Commit message: initial PCB layout is done
Connections:
- net VIN_CONN: now reaches D901.1 (K), J901.1 (Pin_1)
- net VIN_FUSE: now reaches D901.2 (A), F901.1
Other:
- moved on the sheet: D901, F901, J901
Changed lines of the file:
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@@
   (junction (at 127 83.185) (diameter 0) (color 0 0 0 0)
   )
-  (no_connect (at 102.87 85.725))
+  (no_connect (at 85.09 85.725))
   (no_connect (at 164.465 73.025))
   (no_connect (at 153.035 73.025))
@@
     (stroke (width 0) (type default) (color 0 0 0 0))
   )
-  (wire (pts (xy 93.98 80.645) (xy 102.87 80.645))
+  (wire (pts (xy 68.58 80.645) (xy 85.09 80.645))
     (stroke (width 0) (type default) (color 0 0 0 0))
   )
@@
     (stroke (width 0) (type default) (color 0 0 0 0))
   )
-  (wire (pts (xy 93.98 83.185) (xy 95.885 83.185))
+  (wire (pts (xy 68.58 83.185) (xy 70.485 83.185))
     (stroke (width 0) (type default) (color 0 0 0 0))
   )
@@
     (stroke (width 0) (type default) (color 0 0 0 0))
   )
-  (wire (pts (xy 113.03 83.185) (xy 115.57 83.185))
+  (wire (pts (xy 95.25 83.185) (xy 117.475 83.185))
     (stroke (width 0) (type default) (color 0 0 0 0))
   )
@@
     (stroke (width 0) (type default) (color 0 0 0 0))
   )
-  (wire (pts (xy 95.885 83.185) (xy 95.885 85.09))
+  (wire (pts (xy 70.485 83.185) (xy 70.485 85.09))
     (stroke (width 0) (type default) (color 0 0 0 0))
   )
@@
     (stroke (width 0) (type default) (color 0 0 0 0))
   )
-  (wire (pts (xy 123.19 83.185) (xy 127 83.185))
+  (wire (pts (xy 125.095 83.185) (xy 127 83.185))
     (stroke (width 0) (type default) (color 0 0 0 0))
   )
@@
   (wire (pts (xy 127 83.185) (xy 127 74.93))
     (stroke (width 0) (type default) (color 0 0 0 0))
+  )
+  (label "VIN_CONN" (at 71.755 80.645 0)
+    (effects (font (size 1.27 1.27)) (justify left bottom))
+  )
+  (label "VIN_FUSE" (at 104.775 83.185 0)
+    (effects (font (size 1.27 1.27)) (justify left bottom))
   )
   (hierarchical_label "V_IN" (shape input) (at 127 74.93 90)
@@
     (effects (font (size 1.27 1.27)) (justify left))
   )
-  (symbol (lib_id "Device:D_Schottky_Dual_CommonCathode_AAK_Parallel") (at 107.95 83.185 0) (unit 1)
+  (symbol (lib_id "Device:D_Schottky_Dual_CommonCathode_AAK_Parallel") (at 90.17 83.185 0) (unit 1)
     (in_bom yes) (on_board yes)
-    (property "Reference" "D901" (id 0) (at 107.8865 73.66 0))
-    (property "Value" "D_Schottky_Dual_CommonCathode_AAK" (id 1) (at 107.315 107.95 90))
-    (property "Footprint" "Package_TO_SOT_THT:TO-220-3_Vertical" (id 2) (at 109.22 83.185 0)
-      (effects (font (size 1.27 1.27)) hide)
-    )
-    (property "Datasheet" "~" (id 3) (at 109.22 83.185 0)
+    (property "Reference" "D901" (id 0) (at 90.1065 73.66 0))
+    (property "Value" "D_Schottky_Dual_CommonCathode_AAK" (id 1) (at 89.535 107.95 90))
+    (property "Footprint" "Package_TO_SOT_THT:TO-220-3_Vertical" (id 2) (at 91.44 83.185 0)
+      (effects (font (size 1.27 1.27)) hide)
+    )
+    (property "Datasheet" "~" (id 3) (at 91.44 83.185 0)
       (effects (font (size 1.27 1.27)) hide)
     )
@@
     (pin "1")
   )
-  (symbol (lib_id "Connector:Screw_Terminal_01x02") (at 88.9 80.645 0) (mirror y) (unit 1)
+  (symbol (lib_id "Connector:Screw_Terminal_01x02") (at 63.5 80.645 0) (mirror y) (unit 1)
     (in_bom yes) (on_board yes)
-    (property "Reference" "J901" (id 0) (at 83.185 81.915 90))
-    (property "Value" "Screw_Terminal_01x02" (id 1) (at 85.725 81.915 90))
-    (property "Footprint" "TerminalBlock:TerminalBlock_Altech_AK300-2_P5.00mm" (id 2) (at 88.9 80.645 0)
-      (effects (font (size 1.27 1.27)) hide)
-    )
-    (property "Datasheet" "~" (id 3) (at 88.9 80.645 0)
-      (effects (font (size 1.27 1.27)) hide)
-    )
-    (pin "1")
-    (pin "2")
-  )
-  (symbol (lib_id "Device:Fuse") (at 119.38 83.185 90) (unit 1)
-    (in_bom yes) (on_board yes) (fields_autoplaced)
-    (property "Reference" "F901" (id 0) (at 119.38 76.835 90))
-    (property "Value" "Fuse" (id 1) (at 119.38 79.375 90))
-    (property "Footprint" "Fuse:Fuse_Bourns_MF-RHT1000" (id 2) (at 119.38 84.963 90)
-      (effects (font (size 1.27 1.27)) hide)
-    )
-    (property "Datasheet" "~" (id 3) (at 119.38 83.185 0)
+    (property "Reference" "J901" (id 0) (at 57.785 81.915 90))
+    (property "Value" "Screw_Terminal_01x02" (id 1) (at 60.325 81.915 90))
+    (property "Footprint" "TerminalBlock:TerminalBlock_Altech_AK300-2_P5.00mm" (id 2) (at 63.5 80.645 0)
+      (effects (font (size 1.27 1.27)) hide)
+    )
+    (property "Datasheet" "~" (id 3) (at 63.5 80.645 0)
+      (effects (font (size 1.27 1.27)) hide)
+    )
+    (pin "1")
+    (pin "2")
+  )
+  (symbol (lib_id "Device:Fuse") (at 121.285 83.185 90) (unit 1)
+    (in_bom yes) (on_board yes) (fields_autoplaced)
+    (property "Reference" "F901" (id 0) (at 121.285 76.835 90))
+    (property "Value" "Fuse" (id 1) (at 121.285 79.375 90))
+    (property "Footprint" "Fuse:Fuse_Bourns_MF-RHT1000" (id 2) (at 121.285 84.963 90)
+      (effects (font (size 1.27 1.27)) hide)
+    )
+    (property "Datasheet" "~" (id 3) (at 121.285 83.185 0)
       (effects (font (size 1.27 1.27)) hide)
     )
@@
     (pin "2")
   )
-  (symbol (lib_id "power:GND") (at 95.885 85.09 0) (mirror y) (unit 1)
-    (in_bom yes) (on_board yes) (fields_autoplaced)
-    (property "Reference" "#PWR0901" (id 0) (at 95.885 91.44 0)
-      (effects (font (size 1.27 1.27)) hide)
-    )
-    (property "Value" "GND" (id 1) (at 95.885 90.17 0))
-    (property "Footprint" "" (id 2) (at 95.885 85.09 0)
-      (effects (font (size 1.27 1.27)) hide)
-    )
-    (property "Datasheet" "" (id 3) (at 95.885 85.09 0)
-      (effects (font (size 1.27 1.27)) hide)
-    )
+  (symbol (lib_id "power:GND") (at 70.485 85.09 0) (mirror y) (unit 1)
+    (in_bom yes) (on_board yes) (fields_autoplaced)
+    (property "Reference" "#PWR0901" (id 0) (at 70.485 91.44 0)
+      (effects (font (size 1.27 1.27)) hide)
+    )
+    (property "Value" "GND" (id 1) (at 70.485 90.17 0))
+    (property "Footprint" "" (id 2) (at 70.485 85.09 0)
+      (effects (font (size 1.27 1.27)) hide)
+    )
+    (property "Datasheet" "" (id 3) (at 70.485 85.09 0)
+      (effects (font (size 1.27 1.27)) hide)
+    )
