File: Serwo.kicad_sch (KiCad schematic)
At the start: 3 parts, among them J401 Conn_01x03_Male

Commit message: update plików
Other:
- company: (none) -> Szymon Przybył
- title: (none) -> Serwo connector
Changed lines of the file:
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@@
 (kicad_sch (version 20211123) (generator eeschema)
   (paper "A4")
+  (title_block
+    (title "Serwo connector")
+    (date "2023-02-20")
+    (company "Szymon Przybył")
+  )
   (wire (pts (xy 146.05 94.615) (xy 146.05 95.885))
     (stroke (width 0) (type default) (color 0 0 0 0))
