File: Buttons.kicad_sch (KiCad schematic)
At the start: 0 parts

Commit message: update plików
Other:
- company: (none) -> Szymon Przybył
Changed lines of the file:
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@@
 (kicad_sch (version 20211123) (generator eeschema)
   (paper "A4")
+  (title_block
+    (date "2023-02-20")
+    (company "Szymon Przybył")
+  )
   (wire (pts (xy 122.555 75.565) (xy 149.225 75.565))
     (stroke (width 0) (type default) (color 0 0 0 0))
