File: Tensee.kicad_sch (KiCad schematic)
At the start: 1 part, among them IC201 TEENSY_4.1

Commit message: [FEAT] schematic and alyout finished but need to be revieved
Connections:
- net TX1_NC: now reaches IC201.1 (TX1)
- net A0_NC: now reaches IC201.14 (A0)
- net A1_NC: now reaches IC201.15 (A1)
- net A6_NC: now reaches IC201.20 (A6)
- net A7_NC: now reaches IC201.21 (A7)
- net A8_NC: now reaches IC201.22 (A8)
- net A9_NC: now reaches IC201.23 (A9)
- net A10_NC: now reaches IC201.24 (A10)
- net A11_NC: now reaches IC201.25 (A11)
- net A15_NC: now reaches IC201.39 (A15)
- net PROGRAM_NC: now reaches IC201.46 (PROGRAM)
- net ON_OFF_NC: now reaches IC201.47 (ON/OFF)
- net D+_NC: now reaches IC201.50 (D+)
- net D-_NC: now reaches IC201.51 (D-)
- net VIN_NC: now reaches IC201.55 (VIN_(3.6_TO_5.5_VOLTS))
- net RX1_NC: now reaches IC201.57 (RX1)
- net VUSB_NC: now reaches IC201.68 (VUSB)
- net RX2_NC: now reaches IC201.7 (RX2)
- net TX2_NC: now reaches IC201.8 (TX2)
Changed lines of the file:
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@@
     (stroke (width 0) (type default) (color 0 0 0 0))
   )
+  (wire (pts (xy 48.26 102.235) (xy 71.755 102.235))
+    (stroke (width 0) (type default) (color 0 0 0 0))
+  )
   (wire (pts (xy 130.175 94.615) (xy 125.095 94.615))
     (stroke (width 0) (type default) (color 0 0 0 0))
@@
     (stroke (width 0) (type default) (color 0 0 0 0))
   )
+  (wire (pts (xy 48.26 140.335) (xy 71.755 140.335))
+    (stroke (width 0) (type default) (color 0 0 0 0))
+  )
   (wire (pts (xy 63.5 117.475) (xy 71.755 117.475))
     (stroke (width 0) (type default) (color 0 0 0 0))
   )
+  (wire (pts (xy 125.095 147.955) (xy 146.05 147.955))
+    (stroke (width 0) (type default) (color 0 0 0 0))
+  )
   (wire (pts (xy 128.27 122.555) (xy 128.27 130.175))
     (stroke (width 0) (type default) (color 0 0 0 0))
@@
     (stroke (width 0) (type default) (color 0 0 0 0))
   )
+  (wire (pts (xy 125.095 145.415) (xy 146.05 145.415))
+    (stroke (width 0) (type default) (color 0 0 0 0))
+  )
   (wire (pts (xy 130.175 86.995) (xy 125.095 86.995))
     (stroke (width 0) (type default) (color 0 0 0 0))
@@
     (stroke (width 0) (type default) (color 0 0 0 0))
   )
+  (wire (pts (xy 48.26 86.995) (xy 71.755 86.995))
+    (stroke (width 0) (type default) (color 0 0 0 0))
+  )
   (wire (pts (xy 63.5 155.575) (xy 71.755 155.575))
     (stroke (width 0) (type default) (color 0 0 0 0))
@@
     (stroke (width 0) (type default) (color 0 0 0 0))
   )
+  (wire (pts (xy 48.26 145.415) (xy 71.755 145.415))
+    (stroke (width 0) (type default) (color 0 0 0 0))
+  )
+  (wire (pts (xy 125.095 135.255) (xy 146.05 135.255))
+    (stroke (width 0) (type default) (color 0 0 0 0))
+  )
   (wire (pts (xy 125.095 114.935) (xy 128.27 114.935))
     (stroke (width 0) (type default) (color 0 0 0 0))
   )
+  (wire (pts (xy 48.26 147.955) (xy 71.755 147.955))
+    (stroke (width 0) (type default) (color 0 0 0 0))
+  )
   (wire (pts (xy 125.095 112.395) (xy 138.43 112.395))
     (stroke (width 0) (type default) (color 0 0 0 0))
   )
+  (wire (pts (xy 125.095 137.795) (xy 146.05 137.795))
+    (stroke (width 0) (type default) (color 0 0 0 0))
+  )
   (wire (pts (xy 63.5 94.615) (xy 71.755 94.615))
     (stroke (width 0) (type default) (color 0 0 0 0))
@@
     (stroke (width 0) (type default) (color 0 0 0 0))
   )
+  (wire (pts (xy 125.095 107.315) (xy 130.81 107.315))
+    (stroke (width 0) (type default) (color 0 0 0 0))
+  )
   (wire (pts (xy 125.095 120.015) (xy 128.27 120.015))
     (stroke (width 0) (type default) (color 0 0 0 0))
@@
     (stroke (width 0) (type default) (color 0 0 0 0))
   )
+  (wire (pts (xy 125.095 127.635) (xy 135.89 127.635))
+    (stroke (width 0) (type default) (color 0 0 0 0))
+  )
   (wire (pts (xy 63.5 99.695) (xy 71.755 99.695))
     (stroke (width 0) (type default) (color 0 0 0 0))
@@
     (stroke (width 0) (type default) (color 0 0 0 0))
   )
+  (wire (pts (xy 48.26 142.875) (xy 71.755 142.875))
+    (stroke (width 0) (type default) (color 0 0 0 0))
+  )
   (wire (pts (xy 138.43 102.235) (xy 125.095 102.235))
     (stroke (width 0) (type default) (color 0 0 0 0))
@@
     (stroke (width 0) (type default) (color 0 0 0 0))
   )
+  (wire (pts (xy 48.26 135.255) (xy 71.755 135.255))
+    (stroke (width 0) (type default) (color 0 0 0 0))
+  )
   (wire (pts (xy 139.7 142.875) (xy 139.7 141.605))
     (stroke (width 0) (type default) (color 0 0 0 0))
   )
+  (wire (pts (xy 125.095 150.495) (xy 146.05 150.495))
+    (stroke (width 0) (type default) (color 0 0 0 0))
+  )
   (wire (pts (xy 125.095 155.575) (xy 127.635 155.575))
     (stroke (width 0) (type default) (color 0 0 0 0))
@@
     (stroke (width 0) (type default) (color 0 0 0 0))
   )
+  (wire (pts (xy 125.095 125.095) (xy 135.89 125.095))
+    (stroke (width 0) (type default) (color 0 0 0 0))
+  )
+  (wire (pts (xy 48.26 122.555) (xy 71.755 122.555))
+    (stroke (width 0) (type default) (color 0 0 0 0))
+  )
+  (wire (pts (xy 48.26 120.015) (xy 71.755 120.015))
+    (stroke (width 0) (type default) (color 0 0 0 0))
+  )
   (wire (pts (xy 138.43 99.695) (xy 125.095 99.695))
     (stroke (width 0) (type default) (color 0 0 0 0))
@@
     (stroke (width 0) (type default) (color 0 0 0 0))
   )
+  (wire (pts (xy 48.26 137.795) (xy 71.755 137.795))
+    (stroke (width 0) (type default) (color 0 0 0 0))
+  )
   (wire (pts (xy 128.27 120.015) (xy 128.27 114.935))
     (stroke (width 0) (type default) (color 0 0 0 0))
@@
     (stroke (width 0) (type default) (color 0 0 0 0))
   )
+  (wire (pts (xy 48.26 104.775) (xy 71.755 104.775))
+    (stroke (width 0) (type default) (color 0 0 0 0))
+  )
   (wire (pts (xy 125.095 130.175) (xy 128.27 130.175))
     (stroke (width 0) (type default) (color 0 0 0 0))
@@
     (effects (font (size 1.27 1.27)) (justify right))
   )
+  (hierarchical_label "A8_NC" (shape input) (at 48.26 140.335 180)
+    (effects (font (size 1.27 1.27)) (justify right))
+  )
   (hierarchical_label "GPS_RX" (shape input) (at 130.175 94.615 0)
     (effects (font (size 1.27 1.27)) (justify left))
   )
+  (hierarchical_label "VUSB_NC" (shape input) (at 146.05 150.495 0)
+    (effects (font (size 1.27 1.27)) (justify left))
+  )
   (hierarchical_label "DISP_CS" (shape input) (at 63.5 109.855 180)
     (effects (font (size 1.27 1.27)) (justify right))
@@
     (effects (font (size 1.27 1.27)) (justify right))
   )
+  (hierarchical_label "ON_OFF_NC" (shape input) (at 135.89 127.635 0)
+    (effects (font (size 1.27 1.27)) (justify left))
+  )
+  (hierarchical_label "PROGRAM_NC" (shape input) (at 135.89 125.095 0)
+    (effects (font (size 1.27 1.27)) (justify left))
+  )
+  (hierarchical_label "D-_NC" (shape input) (at 146.05 137.795 0)
+    (effects (font (size 1.27 1.27)) (justify left))
+  )
+  (hierarchical_label "A9_NC" (shape input) (at 48.26 142.875 180)
+    (effects (font (size 1.27 1.27)) (justify right))
+  )
+  (hierarchical_label "A1_NC" (shape input) (at 48.26 122.555 180)
+    (effects (font (size 1.27 1.27)) (justify right))
+  )
   (hierarchical_label "BUTTON_B" (shape input) (at 63.5 153.035 180)
     (effects (font (size 1.27 1.27)) (justify right))
   )
+  (hierarchical_label "D+_NC" (shape input) (at 146.05 135.255 0)
+    (effects (font (size 1.27 1.27)) (justify left))
+  )
   (hierarchical_label "ENCODER_A" (shape input) (at 130.175 89.535 0)
     (effects (font (size 1.27 1.27)) (justify left))
@@
     (effects (font (size 1.27 1.27)) (justify left))
   )
+  (hierarchical_label "A11_NC" (shape input) (at 48.26 147.955 180)
+    (effects (font (size 1.27 1.27)) (justify right))
+  )
   (hierarchical_label "ULTRAD3_B" (shape input) (at 63.5 92.075 180)
     (effects (font (size 1.27 1.27)) (justify right))
   )
+  (hierarchical_label "VIN_NC" (shape input) (at 146.05 145.415 0)
+    (effects (font (size 1.27 1.27)) (justify left))
+  )
   (hierarchical_label "GPS_EN" (shape input) (at 130.175 104.775 0)
     (effects (font (size 1.27 1.27)) (justify left))
   )
+  (hierarchical_label "RX1_NC" (shape input) (at 146.05 147.955 0)
+    (effects (font (size 1.27 1.27)) (justify left))
+  )
   (hierarchical_label "CAMERA_SERWO_B" (shape input) (at 63.5 97.155 180)
     (effects (font (size 1.27 1.27)) (justify right))
   )
+  (hierarchical_label "RX2_NC" (shape input) (at 48.26 102.235 180)
+    (effects (font (size 1.27 1.27)) (justify right))
+  )
   (hierarchical_label "DISP_MOSI" (shape input) (at 63.5 112.395 180)
     (effects (font (size 1.27 1.27)) (justify right))
@@
     (effects (font (size 1.27 1.27)) (justify right))
   )
+  (hierarchical_label "A0_NC" (shape input) (at 48.26 120.015 180)
+    (effects (font (size 1.27 1.27)) (justify right))
+  )
+  (hierarchical_label "A7_NC" (shape input) (at 48.26 137.795 180)
+    (effects (font (size 1.27 1.27)) (justify right))
+  )
+  (hierarchical_label "TX1_NC" (shape input) (at 48.26 86.995 180)
+    (effects (font (size 1.27 1.27)) (justify right))
+  )
   (hierarchical_label "BUTTON_A" (shape input) (at 63.5 150.495 180)
     (effects (font (size 1.27 1.27)) (justify right))
@@
     (effects (font (size 1.27 1.27)) (justify right))
   )
+  (hierarchical_label "TX2_NC" (shape input) (at 48.26 104.775 180)
+    (effects (font (size 1.27 1.27)) (justify right))
+  )
   (hierarchical_label "TOF_SCL" (shape input) (at 62.23 132.715 180)
     (effects (font (size 1.27 1.27)) (justify right))
   )
+  (hierarchical_label "A10_NC" (shape input) (at 48.26 145.415 180)
+    (effects (font (size 1.27 1.27)) (justify right))
+  )
   (hierarchical_label "SPEED" (shape input) (at 63.5 99.695 180)
     (effects (font (size 1.27 1.27)) (justify right))
@@
     (effects (font (size 1.27 1.27)) (justify left))
   )
+  (hierarchical_label "A15_NC" (shape input) (at 130.81 107.315 0)
+    (effects (font (size 1.27 1.27)) (justify left))
+  )
   (hierarchical_label "ULTRAD1_B" (shape input) (at 138.43 99.695 0)
     (effects (font (size 1.27 1.27)) (justify left))
@@
     (effects (font (size 1.27 1.27)) (justify right))
   )
+  (hierarchical_label "A6_NC" (shape input) (at 48.26 135.255 180)
+    (effects (font (size 1.27 1.27)) (justify right))
+  )

Commit message: update plików
Connections:
- net VIN_NC is gone; now on net +5V: IC201.55 (VIN_(3.6_TO_5.5_VOLTS))
- net +3.3V: no longer IC201.53 (3.3V_(250_M_A_MAX))
- net +5V: no longer IC201.52 (+5V)
- net A8_NC renamed STEERING1
- net A9_NC renamed STEERING2
- net SPEED renamed SPEED1
- net STEERING renamed SPEED2
- no-connect marks 0 -> 2
Other:
- company: (none) -> Szymon Przybył
- title: (none) -> Tensee
Changed lines of the file:
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@@
 (kicad_sch (version 20211123) (generator eeschema)
   (paper "A4")
+  (title_block
+    (title "Tensee")
+    (date "2023-02-20")
+    (company "Szymon Przybył")
+  )
   (junction (at 127.635 155.575) (diameter 0) (color 0 0 0 0)
   )
@@
   (junction (at 128.27 130.175) (diameter 0) (color 0 0 0 0)
   )
+  (no_connect (at 125.095 140.335))
+  (no_connect (at 125.095 142.875))
   (wire (pts (xy 125.095 109.855) (xy 138.43 109.855))
     (stroke (width 0) (type default) (color 0 0 0 0))
@@
     (stroke (width 0) (type default) (color 0 0 0 0))
   )
-  (wire (pts (xy 125.095 140.335) (xy 134.62 140.335))
-    (stroke (width 0) (type default) (color 0 0 0 0))
-  )
   (wire (pts (xy 161.29 132.715) (xy 161.29 134.62))
     (stroke (width 0) (type default) (color 0 0 0 0))
@@
     (stroke (width 0) (type default) (color 0 0 0 0))
   )
-  (wire (pts (xy 134.62 140.335) (xy 134.62 139.065))
+  (wire (pts (xy 141.605 145.415) (xy 141.605 144.145))
     (stroke (width 0) (type default) (color 0 0 0 0))
   )
-  (wire (pts (xy 48.26 140.335) (xy 71.755 140.335))
+  (wire (pts (xy 62.23 140.335) (xy 71.755 140.335))
     (stroke (width 0) (type default) (color 0 0 0 0))
   )
@@
     (stroke (width 0) (type default) (color 0 0 0 0))
   )
-  (wire (pts (xy 125.095 145.415) (xy 146.05 145.415))
+  (wire (pts (xy 125.095 145.415) (xy 141.605 145.415))
     (stroke (width 0) (type default) (color 0 0 0 0))
   )
@@
     (stroke (width 0) (type default) (color 0 0 0 0))
   )
-  (wire (pts (xy 48.26 142.875) (xy 71.755 142.875))
+  (wire (pts (xy 62.23 142.875) (xy 71.755 142.875))
     (stroke (width 0) (type default) (color 0 0 0 0))
   )
@@
     (stroke (width 0) (type default) (color 0 0 0 0))
   )
-  (wire (pts (xy 139.7 142.875) (xy 139.7 141.605))
-    (stroke (width 0) (type default) (color 0 0 0 0))
-  )
   (wire (pts (xy 125.095 150.495) (xy 146.05 150.495))
     (stroke (width 0) (type default) (color 0 0 0 0))
@@
     (stroke (width 0) (type default) (color 0 0 0 0))
   )
-  (wire (pts (xy 125.095 142.875) (xy 139.7 142.875))
-    (stroke (width 0) (type default) (color 0 0 0 0))
-  )
   (wire (pts (xy 161.29 114.935) (xy 161.29 108.585))
     (stroke (width 0) (type default) (color 0 0 0 0))
@@
     (effects (font (size 1.27 1.27)) (justify right))
   )
-  (hierarchical_label "A8_NC" (shape input) (at 48.26 140.335 180)
-    (effects (font (size 1.27 1.27)) (justify right))
-  )
   (hierarchical_label "GPS_RX" (shape input) (at 130.175 94.615 0)
     (effects (font (size 1.27 1.27)) (justify left))
   )
+  (hierarchical_label "STEERING2" (shape input) (at 62.23 142.875 180)
+    (effects (font (size 1.27 1.27)) (justify right))
+  )
   (hierarchical_label "VUSB_NC" (shape input) (at 146.05 150.495 0)
     (effects (font (size 1.27 1.27)) (justify left))
@@
     (effects (font (size 1.27 1.27)) (justify left))
   )
-  (hierarchical_label "A9_NC" (shape input) (at 48.26 142.875 180)
-    (effects (font (size 1.27 1.27)) (justify right))
-  )
   (hierarchical_label "A1_NC" (shape input) (at 48.26 122.555 180)
     (effects (font (size 1.27 1.27)) (justify right))
@@
     (effects (font (size 1.27 1.27)) (justify right))
   )
-  (hierarchical_label "VIN_NC" (shape input) (at 146.05 145.415 0)
-    (effects (font (size 1.27 1.27)) (justify left))
-  )
   (hierarchical_label "GPS_EN" (shape input) (at 130.175 104.775 0)
     (effects (font (size 1.27 1.27)) (justify left))
@@
     (effects (font (size 1.27 1.27)) (justify right))
   )
+  (hierarchical_label "STEERING1" (shape input) (at 62.23 140.335 180)
+    (effects (font (size 1.27 1.27)) (justify right))
+  )
   (hierarchical_label "ULTRAD2_A" (shape input) (at 63.5 160.655 180)
     (effects (font (size 1.27 1.27)) (justify right))
@@
     (effects (font (size 1.27 1.27)) (justify right))
   )
-  (hierarchical_label "SPEED" (shape input) (at 63.5 99.695 180)
+  (hierarchical_label "SPEED1" (shape input) (at 63.5 99.695 180)
     (effects (font (size 1.27 1.27)) (justify right))
   )
@@
     (effects (font (size 1.27 1.27)) (justify left))
   )
+  (hierarchical_label "SPEED2" (shape input) (at 63.5 107.315 180)
+    (effects (font (size 1.27 1.27)) (justify right))
+  )
   (hierarchical_label "ENCODER_B" (shape input) (at 130.175 92.075 0)
     (effects (font (size 1.27 1.27)) (justify left))
@@
     (effects (font (size 1.27 1.27)) (justify right))
   )
-  (hierarchical_label "STEERING" (shape input) (at 63.5 107.315 180)
-    (effects (font (size 1.27 1.27)) (justify right))
-  )
   (hierarchical_label "ULTRAD2_B" (shape input) (at 130.175 86.995 0)
     (effects (font (size 1.27 1.27)) (justify left))
@@
     (effects (font (size 1.27 1.27)) (justify left))
   )
-  (symbol (lib_id "power:+3.3V") (at 139.7 141.605 0) (unit 1)
+  (symbol (lib_id "power:+5V") (at 141.605 144.145 0) (unit 1)
     (in_bom yes) (on_board yes) (fields_autoplaced)
-    (property "Reference" "#PWR0203" (id 0) (at 139.7 145.415 0)
+    (property "Reference" "#PWR0202" (id 0) (at 141.605 147.955 0)
       (effects (font (size 1.27 1.27)) hide)
     )
-    (property "Value" "+3.3V" (id 1) (at 139.7 136.525 0))
-    (property "Footprint" "" (id 2) (at 139.7 141.605 0)
+    (property "Value" "+5V" (id 1) (at 141.605 138.43 0))
+    (property "Footprint" "" (id 2) (at 141.605 144.145 0)
       (effects (font (size 1.27 1.27)) hide)
     )
-    (property "Datasheet" "" (id 3) (at 139.7 141.605 0)
+    (property "Datasheet" "" (id 3) (at 141.605 144.145 0)
       (effects (font (size 1.27 1.27)) hide)
     )
@@
   (symbol (lib_id "power:GND") (at 161.29 134.62 0) (unit 1)
     (in_bom yes) (on_board yes) (fields_autoplaced)
-    (property "Reference" "#PWR0205" (id 0) (at 161.29 140.97 0)
+    (property "Reference" "#PWR0204" (id 0) (at 161.29 140.97 0)
       (effects (font (size 1.27 1.27)) hide)
     )
@@
     (pin "1")
   )
-  (symbol (lib_id "power:+5V") (at 134.62 139.065 0) (unit 1)
-    (in_bom yes) (on_board yes) (fields_autoplaced)
-    (property "Reference" "#PWR0202" (id 0) (at 134.62 142.875 0)
-      (effects (font (size 1.27 1.27)) hide)
-    )
-    (property "Value" "+5V" (id 1) (at 134.62 133.35 0))
-    (property "Footprint" "" (id 2) (at 134.62 139.065 0)
-      (effects (font (size 1.27 1.27)) hide)
-    )
-    (property "Datasheet" "" (id 3) (at 134.62 139.065 0)
-      (effects (font (size 1.27 1.27)) hide)
-    )
-    (pin "1")
-  )
   (symbol (lib_id "power:+3.3V") (at 161.29 108.585 0) (unit 1)
     (in_bom yes) (on_board yes) (fields_autoplaced)
-    (property "Reference" "#PWR0204" (id 0) (at 161.29 112.395 0)
+    (property "Reference" "#PWR0203" (id 0) (at 161.29 112.395 0)
       (effects (font (size 1.27 1.27)) hide)
     )

Commit message: schematic update after meeting
Connections:
- net +3.3V: no longer names the net of IC201.42 (3.3V_1)
- net +3.3V: no longer IC201.44 (3.3V_2)
- net VOLTMETER renamed A16_NC
- no-connect marks 2 -> 5
Changed lines of the file:
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@@
   (junction (at 128.27 132.715) (diameter 0) (color 0 0 0 0)
   )
-  (junction (at 128.27 114.935) (diameter 0) (color 0 0 0 0)
-  )
   (junction (at 128.27 130.175) (diameter 0) (color 0 0 0 0)
   )
   (no_connect (at 125.095 140.335))
   (no_connect (at 125.095 142.875))
-  (wire (pts (xy 125.095 109.855) (xy 138.43 109.855))
-    (stroke (width 0) (type default) (color 0 0 0 0))
-  )
+  (no_connect (at 125.095 114.935))
+  (no_connect (at 125.095 120.015))
+  (no_connect (at 125.095 117.475))
   (wire (pts (xy 63.5 109.855) (xy 71.755 109.855))
     (stroke (width 0) (type default) (color 0 0 0 0))
@@
     (stroke (width 0) (type default) (color 0 0 0 0))
   )
-  (wire (pts (xy 125.095 114.935) (xy 128.27 114.935))
-    (stroke (width 0) (type default) (color 0 0 0 0))
-  )
   (wire (pts (xy 48.26 147.955) (xy 71.755 147.955))
     (stroke (width 0) (type default) (color 0 0 0 0))
@@
     (stroke (width 0) (type default) (color 0 0 0 0))
   )
-  (wire (pts (xy 128.27 114.935) (xy 161.29 114.935))
-    (stroke (width 0) (type default) (color 0 0 0 0))
-  )
   (wire (pts (xy 63.5 153.035) (xy 71.755 153.035))
     (stroke (width 0) (type default) (color 0 0 0 0))
@@
     (stroke (width 0) (type default) (color 0 0 0 0))
   )
-  (wire (pts (xy 125.095 107.315) (xy 130.81 107.315))
-    (stroke (width 0) (type default) (color 0 0 0 0))
-  )
-  (wire (pts (xy 125.095 120.015) (xy 128.27 120.015))
+  (wire (pts (xy 125.095 107.315) (xy 130.175 107.315))
     (stroke (width 0) (type default) (color 0 0 0 0))
   )
@@
     (stroke (width 0) (type default) (color 0 0 0 0))
   )
-  (wire (pts (xy 161.29 114.935) (xy 161.29 108.585))
-    (stroke (width 0) (type default) (color 0 0 0 0))
-  )
   (wire (pts (xy 125.095 125.095) (xy 135.89 125.095))
     (stroke (width 0) (type default) (color 0 0 0 0))
@@
     (stroke (width 0) (type default) (color 0 0 0 0))
   )
-  (wire (pts (xy 128.27 120.015) (xy 128.27 114.935))
+  (wire (pts (xy 62.23 130.175) (xy 71.755 130.175))
     (stroke (width 0) (type default) (color 0 0 0 0))
   )
-  (wire (pts (xy 62.23 130.175) (xy 71.755 130.175))
+  (wire (pts (xy 125.095 109.855) (xy 130.175 109.855))
     (stroke (width 0) (type default) (color 0 0 0 0))
   )
@@
     (effects (font (size 1.27 1.27)) (justify right))
   )
+  (hierarchical_label "A16_NC" (shape input) (at 130.175 109.855 0)
+    (effects (font (size 1.27 1.27)) (justify left))
+  )
   (hierarchical_label "BUTTON_B" (shape input) (at 63.5 153.035 180)
     (effects (font (size 1.27 1.27)) (justify right))
@@
     (effects (font (size 1.27 1.27)) (justify right))
   )
-  (hierarchical_label "VOLTMETER" (shape input) (at 138.43 109.855 0)
-    (effects (font (size 1.27 1.27)) (justify left))
-  )
   (hierarchical_label "A11_NC" (shape input) (at 48.26 147.955 180)
     (effects (font (size 1.27 1.27)) (justify right))
@@
     (effects (font (size 1.27 1.27)) (justify left))
   )
-  (hierarchical_label "A15_NC" (shape input) (at 130.81 107.315 0)
+  (hierarchical_label "A15_NC" (shape input) (at 130.175 107.315 0)
     (effects (font (size 1.27 1.27)) (justify left))
   )
@@
   (symbol (lib_id "power:GND") (at 161.29 134.62 0) (unit 1)
     (in_bom yes) (on_board yes) (fields_autoplaced)
-    (property "Reference" "#PWR0204" (id 0) (at 161.29 140.97 0)
+    (property "Reference" "#PWR0203" (id 0) (at 161.29 140.97 0)
       (effects (font (size 1.27 1.27)) hide)
     )
@@
       (effects (font (size 1.27 1.27)) hide)
     )
-    (pin "1")
-  )
-  (symbol (lib_id "power:+3.3V") (at 161.29 108.585 0) (unit 1)
-    (in_bom yes) (on_board yes) (fields_autoplaced)
-    (property "Reference" "#PWR0203" (id 0) (at 161.29 112.395 0)
-      (effects (font (size 1.27 1.27)) hide)
-    )
-    (property "Value" "+3.3V" (id 1) (at 161.29 103.505 0))
-    (property "Footprint" "" (id 2) (at 161.29 108.585 0)
-      (effects (font (size 1.27 1.27)) hide)
-    )
-    (property "Datasheet" "" (id 3) (at 161.29 108.585 0)
-      (effects (font (size 1.27 1.27)) hide)
-    )
