File: UltraSonicSensorConnector.kicad_sch (KiCad schematic)
At the start: 3 parts, among them J601 Conn_01x04_Male

Commit message: update plików
Parts:
- J601: value Conn_01x04_Male -> JST 2.56mm
Other:
- company: (none) -> Szymon Przybył
- title: (none) -> Ultrasonic sensor connector
Changed lines of the file:
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@@
 (kicad_sch (version 20211123) (generator eeschema)
   (paper "A4")
+  (title_block
+    (title "Ultrasonic sensor connector")
+    (date "2023-02-20")
+    (company "Szymon Przybył")
+  )
   (wire (pts (xy 143.51 102.87) (xy 143.51 104.14))
     (stroke (width 0) (type default) (color 0 0 0 0))
@@
   )
   (symbol (lib_id "Connector:Conn_01x04_Male") (at 137.16 97.79 0) (unit 1)
-    (in_bom yes) (on_board yes) (fields_autoplaced)
-    (property "Reference" "J601" (id 0) (at 135.89 97.7899 0)
-      (effects (font (size 1.27 1.27)) (justify right))
-    )
-    (property "Value" "Conn_01x04_Male" (id 1) (at 135.89 100.3299 0)
-      (effects (font (size 1.27 1.27)) (justify right))
-    )
+    (in_bom yes) (on_board yes)
+    (property "Reference" "J601" (id 0) (at 130.175 97.79 0))
+    (property "Value" "JST 2.56mm" (id 1) (at 130.175 100.33 0))
     (property "Footprint" "Connector_JST:JST_XH_B4B-XH-A_1x04_P2.50mm_Vertical" (id 2) (at 137.16 97.79 0)
       (effects (font (size 1.27 1.27)) hide)
