File: AutkoPcb.kicad_pcb (KiCad board)
At the start: 2 copper layers, 83.8 x 105.5 mm, 60 parts, among them IC201 TEENSY_4.1, J101 JST 2.56mm, J102 JST 2.56mm, J103 JST 2.56mm, J104 JST 2.56mm, J105 JST 2.56mm, J107 JST 2.56mm, J108 JST 2.56mm, J109 JST 2.56mm, J110 JST 2.56mm, J111 JST 2.56mm, J112 JST 2.56mm, J113 JST 2.56mm, J114 Conn_01x12_Pin, J401 Conn_01x03_Male, J501 Conn_01x03_Male, J601 JST 2.56mm, J701 JST 2.56mm, J801 JST 2.56mm, J901 ARK 5mm, J902 Barrel_Jack_MountingPin, J903 Barrel_Jack_MountingPin, J904 ARK 5mm, J905 JST 2.54mm, J906 JST 2.54mm, J907 JST 2.56mm, SW1001 SW_Push, SW1101 SW_Push, SW1201 SW_Push, SW1301 SW_Push, U901 AZ1117-3.3

Commit message: release
Other:
- board text added: "10K"
- board text added: "KARR PCB v1.0 14.02.2023"
- board text added: "SERV"
- board text removed: "CAM_A"
Changed lines of the file:
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@@
       (plot_on_all_layers_selection 0x0000000_00000000)
       (disableapertmacros false)
-      (usegerberextensions false)
+      (usegerberextensions true)
       (usegerberattributes true)
       (usegerberadvancedattributes true)
@@
       (plotinvisibletext false)
       (sketchpadsonfab false)
-      (subtractmaskfromsilk false)
+      (subtractmaskfromsilk true)
       (outputformat 1)
       (mirror false)
-      (drillshape 1)
+      (drillshape 0)
       (scaleselection 1)
-      (outputdirectory "")
+      (outputdirectory "C:/Codes/ISA/karr-pcb/build/")
     )
   )
@@
     (property "ki_keywords" "cap capacitor")
     (attr through_hole)
-    (fp_text reference "C1301" (at 5.25 0 unlocked) (layer "F.SilkS")
+    (fp_text reference "C1301" (at 5.167986 0.748006 unlocked) (layer "F.SilkS")
         (effects (font (size 0.6 0.6) (thickness 0.15)))
     )
@@
         (effects (font (size 1 1) (thickness 0.15)))
     )
-    (fp_text user "EN" (at 12.7 -16.8 180 unlocked) (layer "F.SilkS")
+    (fp_text user "EN" (at 12.7 -16.8 unlocked) (layer "F.SilkS")
         (effects (font (size 1 1) (thickness 0.15)))
     )
-    (fp_text user "VOUT" (at 20.3 -15.7 180 unlocked) (layer "F.SilkS")
+    (fp_text user "VOUT" (at 20.3 -15.7 unlocked) (layer "F.SilkS")
         (effects (font (size 1 1) (thickness 0.15)))
     )
@@
         (effects (font (size 1 1) (thickness 0.15)))
     )
-    (fp_text user "PG" (at 15.3 -16.8 180 unlocked) (layer "F.SilkS")
+    (fp_text user "PG" (at 15.3 -16.8 unlocked) (layer "F.SilkS")
         (effects (font (size 1 1) (thickness 0.15)))
     )
@@
         (effects (font (size 1 1) (thickness 0.15)))
     )
-    (fp_text user "FB" (at 17.8 -16.8 180 unlocked) (layer "F.SilkS")
+    (fp_text user "FB" (at 17.8 -16.8 unlocked) (layer "F.SilkS")
         (effects (font (size 1 1) (thickness 0.15)))
     )
@@
     (property "ki_keywords" "cap capacitor")
     (attr through_hole)
-    (fp_text reference "C1201" (at 5.25 0 unlocked) (layer "F.SilkS")
+    (fp_text reference "C1201" (at 5.20294 0.5018 unlocked) (layer "F.SilkS")
         (effects (font (size 0.6 0.6) (thickness 0.15)))
     )
@@
     (property "ki_keywords" "cap capacitor")
     (attr through_hole)
-    (fp_text reference "C1001" (at 5.66 0.6 180 unlocked) (layer "F.SilkS")
+    (fp_text reference "C1001" (at 5.66 0.6 unlocked) (layer "F.SilkS")
         (effects (font (size 0.6 0.6) (thickness 0.15)))
     )
@@
     (property "ki_keywords" "cap capacitor")
     (attr through_hole)
-    (fp_text reference "C1101" (at 5.2 -0.025 unlocked) (layer "F.SilkS")
+    (fp_text reference "C1101" (at 5.117986 0.498071 unlocked) (layer "F.SilkS")
         (effects (font (size 0.6 0.6) (thickness 0.15)))
     )
@@
     (effects (font (size 0.6 0.6) (thickness 0.15)))
   )
+  (gr_text "KARR PCB v1.0\n14.02.2023" (at 170.447914 129.079784) (layer "F.SilkS")
+    (effects (font (size 1.5 1.5) (thickness 0.2)) (justify left bottom))
+  )
   (gr_text "3.3V" (at 109 64.7 90) (layer "F.SilkS")
     (effects (font (size 0.6 0.6) (thickness 0.15)))
@@
     (effects (font (size 0.6 0.6) (thickness 0.15)))
   )
-  (gr_text "CAM_A" (at 134.1 27.6 90) (layer "F.SilkS")
+  (gr_text "SERV" (at 134.096979 27.763933 90) (layer "F.SilkS")
     (effects (font (size 0.6 0.6) (thickness 0.15)))
   )
@@
     (effects (font (size 0.6 0.6) (thickness 0.15) bold) (justify left bottom))
   )
+  (gr_text "100nF" (at 125.49691 63.191219) (layer "F.SilkS")
+    (effects (font (size 0.6 0.6) (thickness 0.15) bold) (justify left bottom))
+  )
   (gr_text "3.3V" (at 111.5 55.332143 90) (layer "F.SilkS")
     (effects (font (size 0.6 0.6) (thickness 0.15)))
@@
     (effects (font (size 0.6 0.6) (thickness 0.15) bold) (justify left bottom))
   )
+  (gr_text "100nF" (at 125.881408 67.945012) (layer "F.SilkS")
+    (effects (font (size 0.6 0.6) (thickness 0.15) bold) (justify left bottom))
+  )
   (gr_text "A1" (at 186.571428 38.845452) (layer "F.SilkS")
     (effects (font (size 0.6 0.6) (thickness 0.15)))
@@
     (effects (font (size 0.7 0.7) (thickness 0.15) bold) (justify left bottom))
   )
+  (gr_text "10K" (at 127.850556 69.931637) (layer "F.SilkS")
+    (effects (font (size 0.6 0.6) (thickness 0.15) bold) (justify left bottom))
+  )
   (gr_text "GND" (at 123.3 117.7) (layer "F.SilkS")
     (effects (font (size 0.7 0.7) (thickness 0.15) bold) (justify left bottom))
@@
     (effects (font (size 0.6 0.6) (thickness 0.15)))
   )
+  (gr_text "10K" (at 127.816541 65.11489) (layer "F.SilkS")
+    (effects (font (size 0.6 0.6) (thickness 0.15) bold) (justify left bottom))
+  )
   (gr_text "4.7k" (at 178.119912 57.971482 90) (layer "F.SilkS")
     (effects (font (size 0.6 0.6) (thickness 0.15) bold) (justify left bottom))
@@
     (effects (font (size 0.6 0.6) (thickness 0.15)))
   )
+  (gr_text "100nF" (at 125.916363 77.627372) (layer "F.SilkS")
+    (effects (font (size 0.6 0.6) (thickness 0.15) bold) (justify left bottom))
+  )
   (gr_text "3.3V" (at 187 56.6) (layer "F.SilkS")
     (effects (font (size 0.6 0.6) (thickness 0.15)))
@@
     (effects (font (size 0.6 0.6) (thickness 0.15)))
   )
+  (gr_text "10K" (at 127.862207 74.685431) (layer "F.SilkS")
+    (effects (font (size 0.6 0.6) (thickness 0.15) bold) (justify left bottom))
+  )
+  (gr_text "10K" (at 127.908813 60.039552) (layer "F.SilkS")
+    (effects (font (size 0.6 0.6) (thickness 0.15) bold) (justify left bottom))
+  )
   (gr_text "5V IN" (at 162.865075 105.536462 90) (layer "F.SilkS")
     (effects (font (size 0.6 0.6) (thickness 0.15) bold) (justify left bottom))
@@
     (effects (font (size 0.6 0.6) (thickness 0.15)))
   )
+  (gr_text "100nF" (at 125.986271 72.73376) (layer "F.SilkS")
+    (effects (font (size 0.6 0.6) (thickness 0.15) bold) (justify left bottom))
+  )
   (gr_text "EN" (at 168.3 70.099999 90) (layer "F.SilkS")
